Commit message: Improve retargetting by adding constraints penalty

File: data/resources/robots/g1_inspirehands/G1_inspire_hands.urdf (robot description, URDF)
Before this commit: robot g1_29dof_rev_1_0_with_inspire_hand_DFQ, 74 links, 73 joints
Links:
- link L_hand_base_link: geometry collision mesh filename=/home/chenghuailin/hri-retargetting/data/resources/robots/g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; visual mesh filename=/home/chenghuailin/hri-retargetting/data/resources/robots/g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
- link L_index_intermediate: geometry collision mesh filename=/home/chenghuailin/hri-retargetting/data/resources/robots/g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; visual mesh filename=/home/chenghuailin/hri-retargetting/data/resources/robots/g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
- link L_index_proximal: geometry collision mesh filename=/home/chenghuailin/hri-retargetting/data/resources/robots/g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; visual mesh filename=/home/chenghuailin/hri-retargetting/data/resources/robots/g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
- link L_middle_intermediate: geometry collision mesh filename=/home/chenghuailin/hri-retargetting/data/resources/robots/g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; visual mesh filename=/home/chenghuailin/hri-retargetting/data/resources/robots/g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
- link L_middle_proximal: geometry collision mesh filename=/home/chenghuailin/hri-retargetting/data/resources/robots/g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; visual mesh filename=/home/chenghuailin/hri-retargetting/data/resources/robots/g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
- link L_pinky_intermediate: geometry collision mesh filename=/home/chenghuailin/hri-retargetting/data/resources/robots/g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; visual mesh filename=/home/chenghuailin/hri-retargetting/data/resources/robots/g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
- link L_pinky_proximal: geometry collision mesh filename=/home/chenghuailin/hri-retargetting/data/resources/robots/g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; visual mesh filename=/home/chenghuailin/hri-retargetting/data/resources/robots/g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
- link L_ring_intermediate: geometry collision mesh filename=/home/chenghuailin/hri-retargetting/data/resources/robots/g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; visual mesh filename=/home/chenghuailin/hri-retargetting/data/resources/robots/g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
- link L_ring_proximal: geometry collision mesh filename=/home/chenghuailin/hri-retargetting/data/resources/robots/g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; visual mesh filename=/home/chenghuailin/hri-retargetting/data/resources/robots/g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
- link L_thumb_distal: geometry collision mesh filename=/home/chenghuailin/hri-retargetting/data/resources/robots/g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; visual mesh filename=/home/chenghuailin/hri-retargetting/data/resources/robots/g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
- link L_thumb_intermediate: geometry collision mesh filename=/home/chenghuailin/hri-retargetting/data/resources/robots/g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; visual mesh filename=/home/chenghuailin/hri-retargetting/data/resources/robots/g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
- link L_thumb_proximal: geometry collision mesh filename=/home/chenghuailin/hri-retargetting/data/resources/robots/g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; visual mesh filename=/home/chenghuailin/hri-retargetting/data/resources/robots/g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
- link L_thumb_proximal_base: geometry collision mesh filename=/home/chenghuailin/hri-retargetting/data/resources/robots/g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; visual mesh filename=/home/chenghuailin/hri-retargetting/data/resources/robots/g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
- link R_hand_base_link: geometry collision mesh filename=/home/chenghuailin/hri-retargetting/data/resources/robots/g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; visual mesh filename=/home/chenghuailin/hri-retargetting/data/resources/robots/g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
- link R_index_intermediate: geometry collision mesh filename=/home/chenghuailin/hri-retargetting/data/resources/robots/g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; visual mesh filename=/home/chenghuailin/hri-retargetting/data/resources/robots/g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
- link R_index_proximal: geometry collision mesh filename=/home/chenghuailin/hri-retargetting/data/resources/robots/g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; visual mesh filename=/home/chenghuailin/hri-retargetting/data/resources/robots/g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
- link R_middle_intermediate: geometry collision mesh filename=/home/chenghuailin/hri-retargetting/data/resources/robots/g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; visual mesh filename=/home/chenghuailin/hri-retargetting/data/resources/robots/g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
- link R_middle_proximal: geometry collision mesh filename=/home/chenghuailin/hri-retargetting/data/resources/robots/g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; visual mesh filename=/home/chenghuailin/hri-retargetting/data/resources/robots/g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
- link R_pinky_intermediate: geometry collision mesh filename=/home/chenghuailin/hri-retargetting/data/resources/robots/g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; visual mesh filename=/home/chenghuailin/hri-retargetting/data/resources/robots/g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
- link R_pinky_proximal: geometry collision mesh filename=/home/chenghuailin/hri-retargetting/data/resources/robots/g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; visual mesh filename=/home/chenghuailin/hri-retargetting/data/resources/robots/g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
- link R_ring_intermediate: geometry collision mesh filename=/home/chenghuailin/hri-retargetting/data/resources/robots/g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; visual mesh filename=/home/chenghuailin/hri-retargetting/data/resources/robots/g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
- link R_ring_proximal: geometry collision mesh filename=/home/chenghuailin/hri-retargetting/data/resources/robots/g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; visual mesh filename=/home/chenghuailin/hri-retargetting/data/resources/robots/g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
- link R_thumb_distal: geometry collision mesh filename=/home/chenghuailin/hri-retargetting/data/resources/robots/g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; visual mesh filename=/home/chenghuailin/hri-retargetting/data/resources/robots/g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
- link R_thumb_intermediate: geometry collision mesh filename=/home/chenghuailin/hri-retargetting/data/resources/robots/g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; visual mesh filename=/home/chenghuailin/hri-retargetting/data/resources/robots/g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
- link R_thumb_proximal: geometry collision mesh filename=/home/chenghuailin/hri-retargetting/data/resources/robots/g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; visual mesh filename=/home/chenghuailin/hri-retargetting/data/resources/robots/g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
- link R_thumb_proximal_base: geometry collision mesh filename=/home/chenghuailin/hri-retargetting/data/resources/robots/g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; visual mesh filename=/home/chenghuailin/hri-retargetting/data/resources/robots/g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
- link head_link: geometry collision mesh filename=/home/chenghuailin/hri-retargetting/data/resources/robots/g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; visual mesh filename=/home/chenghuailin/hri-retargetting/data/resources/robots/g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
- link left_ankle_pitch_link: geometry collision mesh filename=/home/chenghuailin/hri-retargetting/data/resources/robots/g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; visual mesh filename=/home/chenghuailin/hri-retargetting/data/resources/robots/g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
- link left_ankle_roll_link: geometry collision sphere radius=0.005; collision sphere radius=0.005
- link left_elbow_link: geometry collision mesh filename=/home/chenghuailin/hri-retargetting/data/resources/robots/g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; visual mesh filename=/home/chenghuailin/hri-retargetting/data/resources/robots/g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
- link left_hip_pitch_link: geometry collision mesh filename=/home/chenghuailin/hri-retargetting/data/resources/robots/g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; visual mesh filename=/home/chenghuailin/hri-retargetting/data/resources/robots/g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
- link left_hip_roll_link: geometry collision mesh filename=/home/chenghuailin/hri-retargetting/data/resources/robots/g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; visual mesh filename=/home/chenghuailin/hri-retargetting/data/resources/robots/g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
- link left_hip_yaw_link: geometry collision mesh filename=/home/chenghuailin/hri-retargetting/data/resources/robots/g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; visual mesh filename=/home/chenghuailin/hri-retargetting/data/resources/robots/g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
- link left_knee_link: geometry collision mesh filename=/home/chenghuailin/hri-retargetting/data/resources/robots/g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; visual mesh filename=/home/chenghuailin/hri-retargetting/data/resources/robots/g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
- link left_shoulder_pitch_link: geometry collision cylinder length=0.05 radius=0.03; visual mesh filename=/home/chenghuailin/hri-retargetting/data/resources/robots/g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
- link left_shoulder_roll_link: geometry collision cylinder length=0.03 radius=0.03; visual mesh filename=/home/chenghuailin/hri-retargetting/data/resources/robots/g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
- link left_shoulder_yaw_link: geometry collision mesh filename=/home/chenghuailin/hri-retargetting/data/resources/robots/g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; visual mesh filename=/home/chenghuailin/hri-retargetting/data/resources/robots/g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
- link left_wrist_pitch_link: geometry collision mesh filename=/home/chenghuailin/hri-retargetting/data/resources/robots/g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; visual mesh filename=/home/chenghuailin/hri-retargetting/data/resources/robots/g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
- link left_wrist_roll_link: geometry collision mesh filename=/home/chenghuailin/hri-retargetting/data/resources/robots/g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; visual mesh filename=/home/chenghuailin/hri-retargetting/data/resources/robots/g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
- link left_wrist_yaw_link: geometry collision mesh filename=/home/chenghuailin/hri-retargetting/data/resources/robots/g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; visual mesh filename=/home/chenghuailin/hri-retargetting/data/resources/robots/g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
- link logo_link: geometry collision mesh filename=/home/chenghuailin/hri-retargetting/data/resources/robots/g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; visual mesh filename=/home/chenghuailin/hri-retargetting/data/resources/robots/g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
- link pelvis: geometry visual mesh filename=/home/chenghuailin/hri-retargetting/data/resources/robots/g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
- link pelvis_contour_link: geometry collision mesh filename=/home/chenghuailin/hri-retargetting/data/resources/robots/g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; visual mesh filename=/home/chenghuailin/hri-retargetting/data/resources/robots/g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
- link right_ankle_pitch_link: geometry collision mesh filename=/home/chenghuailin/hri-retargetting/data/resources/robots/g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; visual mesh filename=/home/chenghuailin/hri-retargetting/data/resources/robots/g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
- link right_ankle_roll_link: geometry collision sphere radius=0.005; collision sphere radius=0.005
- link right_elbow_link: geometry collision mesh filename=/home/chenghuailin/hri-retargetting/data/resources/robots/g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; visual mesh filename=/home/chenghuailin/hri-retargetting/data/resources/robots/g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
- link right_hip_pitch_link: geometry collision mesh filename=/home/chenghuailin/hri-retargetting/data/resources/robots/g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; visual mesh filename=/home/chenghuailin/hri-retargetting/data/resources/robots/g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
- link right_hip_roll_link: geometry collision mesh filename=/home/chenghuailin/hri-retargetting/data/resources/robots/g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; visual mesh filename=/home/chenghuailin/hri-retargetting/data/resources/robots/g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
- link right_hip_yaw_link: geometry collision mesh filename=/home/chenghuailin/hri-retargetting/data/resources/robots/g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; visual mesh filename=/home/chenghuailin/hri-retargetting/data/resources/robots/g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
- link right_knee_link: geometry collision mesh filename=/home/chenghuailin/hri-retargetting/data/resources/robots/g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; visual mesh filename=/home/chenghuailin/hri-retargetting/data/resources/robots/g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
- link right_shoulder_pitch_link: geometry collision cylinder length=0.05 radius=0.03; visual mesh filename=/home/chenghuailin/hri-retargetting/data/resources/robots/g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
- link right_shoulder_roll_link: geometry collision cylinder length=0.03 radius=0.03; visual mesh filename=/home/chenghuailin/hri-retargetting/data/resources/robots/g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
- link right_shoulder_yaw_link: geometry collision mesh filename=/home/chenghuailin/hri-retargetting/data/resources/robots/g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; visual mesh filename=/home/chenghuailin/hri-retargetting/data/resources/robots/g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
- link right_wrist_pitch_link: geometry collision mesh filename=/home/chenghuailin/hri-retargetting/data/resources/robots/g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; visual mesh filename=/home/chenghuailin/hri-retargetting/data/resources/robots/g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
- link right_wrist_roll_link: geometry collision mesh filename=/home/chenghuailin/hri-retargetting/data/resources/robots/g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; visual mesh filename=/home/chenghuailin/hri-retargetting/data/resources/robots/g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
- link right_wrist_yaw_link: geometry collision mesh filename=/home/chenghuailin/hri-retargetting/data/resources/robots/g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; visual mesh filename=/home/chenghuailin/hri-retargetting/data/resources/robots/g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
- link torso_link: geometry collision mesh filename=/home/chenghuailin/hri-retargetting/data/resources/robots/g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; visual mesh filename=/home/chenghuailin/hri-retargetting/data/resources/robots/g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
- link waist_roll_link: geometry visual mesh filename=/home/chenghuailin/hri-retargetting/data/resources/robots/g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
- link waist_support_link: geometry collision mesh filename=/home/chenghuailin/hri-retargetting/data/resources/robots/g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; visual mesh filename=/home/chenghuailin/hri-retargetting/data/resources/robots/g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
- link waist_yaw_link: geometry visual mesh filename=/home/chenghuailin/hri-retargetting/data/resources/robots/g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
Joints:
- joint left_shoulder_pitch_joint: limit lower=-3.0892 upper=2.6704 effort=25 velocity=37 -> lower=-3.0892 upper=2.6704 effort=25 velocity=30
